File: pcb/S3-MK1.kicad_sch (KiCad schematic)
At the start: 6 parts, among them J2 SW_420, U1 WEMOS_D1_mini, U2 DHT11

Commit message: journal 4 : added, connected new sym, footprints
Parts:
- added BT1: Battery_Cell, custom_footprints_1:Battery_LiPo_Custom, symbol Device:Battery_Cell
- added BZ1: Buzzer, Buzzer_Beeper:Buzzer_TDK_PS1240P02BT_D12.2mm_H6.5mm, symbol Device:Buzzer
- added D1: NeoPixel_THT, LED_SMD:LED_SK6812_PLCC4_5.0x5.0mm_P3.2mm, symbol LED:NeoPixel_THT
- added R2: R, Resistor_THT:R_Axial_DIN0204_L3.6mm_D1.6mm_P5.08mm_Horizontal, symbol Device:R
- added SW1: SW_Slide_DPDT, Button_Switch_THT:SW_CK_JS202011CQN_DPDT_Straight, symbol Switch:SW_Slide_DPDT
- J1: footprint (none) -> custom_footprints_1:LD2420_custom
- J2: footprint (none) -> custom_footprints_1:Vibration_sensor_SW420_custom
Connections:
- net at A1.1 (VCC): now also J1.1 (VCC), J2.1 (VCC), R1.2, U1.8 (3V3), U2.1 (VDD), BZ1.1 (+), D1.3 (VDD), SW1.4 (A)
- net at A1.2 (GND): now also J1.2 (GND), J2.2 (GND), U1.10 (GND), U2.4 (GND), BT1.2 (-), D1.2 (GND), R2.1
- net at A1.3 (SCL): now also U1.14 (SCL/D1)
- net at A1.4 (SDA): now also U1.13 (SDA/D2)
- net at U1.11 (D4): now also D1.4 (DIN)
- net at U1.12 (D3): now also U2.2 (DATA)
- net at U1.2 (A0): now also R1.1, R2.2
- net at U1.3 (D0): now also BZ1.2 (-)
- net at U1.4 (SCK/D5): now also J1.3 (RX)
- net at U1.5 (MISO/D6): now also J1.4 (Pin_4)
- net at U1.6 (MOSI/D7): now also J2.3 (D0)
- new net: BT1.1 (+), SW1.5 (B)
Other:
- moved on the sheet: R1

Commit message: journal 7 : added new components, firmware
Parts:
- added J3: audio_sensor_custom, symbol custom_s3:audio_sensor_custom
Connections:
- net at A1.1 (VCC), BZ1.1 (+), D1.3 (VDD)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: now also J3.1 (Pin_1)
- net at A1.2 (GND), BT1.2 (-), D1.2 (GND)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: now also J3.2 (Pin_2)
- net at R1.1, R2.2: now also U1.7 (CS/D8); no longer U1.2 (A0)
- new net: J3.3 (Pin_3), U1.2 (A0)
Changed lines of the file:
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@@
+	)
+	(junction
+		(at 130.81 41.91)
+		(diameter 0)
+		(color 0 0 0 0)
 	)
 	(junction
@@
 	(wire
 		(pts
+			(xy 130.81 41.91) (xy 144.78 41.91)
+		)
+		(stroke
+			(width 0)
+			(type default)
+		)
+	)
+	(wire
+		(pts
 			(xy 113.03 68.58) (xy 124.46 68.58)
 		)
@@
 	(wire
 		(pts
+			(xy 123.19 96.52) (xy 102.87 96.52)
+		)
+		(stroke
+			(width 0)
+			(type default)
+		)
+	)
+	(wire
+		(pts
 			(xy 55.88 21.59) (xy 105.41 21.59)
 		)
@@
 	(wire
 		(pts
+			(xy 123.19 78.74) (xy 123.19 96.52)
+		)
+		(stroke
+			(width 0)
+			(type default)
+		)
+	)
+	(wire
+		(pts
 			(xy 105.41 27.94) (xy 105.41 36.83)
 		)
@@
 	(wire
 		(pts
+			(xy 86.36 45.72) (xy 121.92 45.72)
+		)
+		(stroke
+			(width 0)
+			(type default)
+		)
+	)
+	(wire
+		(pts
 			(xy 172.72 80.01) (xy 165.1 80.01)
 		)
@@
 	(wire
 		(pts
+			(xy 133.35 76.2) (xy 130.81 76.2)
+		)
+		(stroke
+			(width 0)
+			(type default)
+		)
+	)
+	(wire
+		(pts
 			(xy 152.4 55.88) (xy 157.48 55.88)
 		)
@@
 	(wire
 		(pts
+			(xy 133.35 78.74) (xy 123.19 78.74)
+		)
+		(stroke
+			(width 0)
+			(type default)
+		)
+	)
+	(wire
+		(pts
 			(xy 115.57 71.12) (xy 113.03 71.12)
 		)
@@
 	(wire
 		(pts
-			(xy 113.03 45.72) (xy 86.36 45.72)
-		)
-		(stroke
-			(width 0)
-			(type default)
-		)
-	)
-	(wire
-		(pts
 			(xy 77.47 67.31) (xy 77.47 64.77)
 		)
@@
 	(wire
 		(pts
+			(xy 129.54 55.88) (xy 129.54 81.28)
+		)
+		(stroke
+			(width 0)
+			(type default)
+		)
+	)
+	(wire
+		(pts
 			(xy 102.87 110.49) (xy 146.05 110.49)
 		)
@@
 	(wire
 		(pts
+			(xy 121.92 45.72) (xy 121.92 78.74)
+		)
+		(stroke
+			(width 0)
+			(type default)
+		)
+	)
+	(wire
+		(pts
 			(xy 138.43 30.48) (xy 132.08 30.48)
 		)
@@
 	(wire
 		(pts
-			(xy 105.41 41.91) (xy 144.78 41.91)
-		)
-		(stroke
-			(width 0)
-			(type default)
-		)
-	)
-	(wire
-		(pts
-			(xy 113.03 55.88) (xy 113.03 45.72)
+			(xy 105.41 41.91) (xy 130.81 41.91)
 		)
 		(stroke
@@
 	(wire
 		(pts
+			(xy 121.92 78.74) (xy 113.03 78.74)
+		)
+		(stroke
+			(width 0)
+			(type default)
+		)
+	)
+	(wire
+		(pts
 			(xy 132.08 30.48) (xy 132.08 19.05)
 		)
@@
 	(wire
 		(pts
+			(xy 130.81 41.91) (xy 130.81 76.2)
+		)
+		(stroke
+			(width 0)
+			(type default)
+		)
+	)
+	(wire
+		(pts
 			(xy 88.9 41.91) (xy 105.41 41.91)
 		)
@@
 		(pts
 			(xy 144.78 48.26) (xy 144.78 41.91)
+		)
+		(stroke
+			(width 0)
+			(type default)
+		)
+	)
+	(wire
+		(pts
+			(xy 129.54 81.28) (xy 133.35 81.28)
+		)
+		(stroke
+			(width 0)
+			(type default)
+		)
+	)
+	(wire
+		(pts
+			(xy 113.03 55.88) (xy 129.54 55.88)
 		)
 		(stroke
@@
 					(unit 1)
 				)
+			)
+		)
+	)
+	(symbol
+		(lib_id "custom_s3:audio_sensor_custom")
+		(at 138.43 78.74 0)
+		(unit 1)
+		(body_style 1)
+		(exclude_from_sim no)
+		(in_bom yes)
+		(on_board yes)
+		(in_pos_files yes)
+		(dnp no)
+		(property "Reference" "J3"
+			(at 143.51 76.8349 0)
+			(show_name no)
+			(do_not_autoplace no)
+			(effects
+				(font
+					(size 1.27 1.27)
+				)
+				(justify left)
+			)
+		)
+		(property "Value" "audio_sensor_custom"
+			(at 135.128 72.136 0)
+			(show_name no)
+			(do_not_autoplace no)
+			(effects
+				(font
+					(size 1.27 1.27)
+				)
+				(justify left)
+			)
+		)
+		(property "Footprint" ""
+			(at 138.43 78.74 0)
+			(hide yes)
+			(show_name no)
+			(do_not_autoplace no)
+			(effects
+				(font
+					(size 1.27 1.27)
+				)
+			)
+		)
+		(property "Datasheet" ""
+			(at 138.43 78.74 0)
+			(hide yes)
+			(show_name no)
+			(do_not_autoplace no)
+			(effects
+				(font
+					(size 1.27 1.27)
+				)
+			)
+		)
+		(property "Description" ""
+			(at 138.43 78.74 0)
+			(hide yes)
+			(show_name no)
+			(do_not_autoplace no)
+			(effects
+				(font
+					(size 1.27 1.27)
+				)
+			)
+		)
+		(pin "3"
+		)
+		(pin "2"
+		)
+		(pin "1"
+		)
+		(instances
+			(project "S3-MK1"
+				(path "/3b160dbc-653e-496a-842f-ecdcc5a2cc2f"
+					(reference "J3")
+					(unit 1)
+				)

Commit message: added journal 8, pcb files, libs
Parts:
- added BT2: Battery_Cell, custom_footprints_1:Battery_LiPo_Custom, symbol Device:Battery_Cell
- added BZ2: Buzzer, Buzzer_Beeper:MagneticBuzzer_Kingstate_KCG0601, symbol Device:Buzzer
- added BZ3: Haptic_Vibration, symbol Device:Buzzer
- added D2: NeoPixel_THT, LED_SMD:LED_SK6812_PLCC4_5.0x5.0mm_P3.2mm, symbol LED:NeoPixel_THT
- added J5: OLED_128x64, ScottoKeebs_Components:OLED_128x64, symbol ScottoKeebs:OLED_128x64
- added SW2: SW_Slide_DPDT, Button_Switch_THT:SW_CK_JS202011CQN_DPDT_Straight, symbol Switch:SW_Slide_DPDT
- added SW3, SW4, SW5, SW6: SW_Push, symbol Switch:SW_Push
- added U3: WEMOS_D1_mini, RF_Module:WEMOS_D1_mini_light, symbol RF_Module:WEMOS_D1_mini
- J3: footprint (none) -> custom_footprints_1:Audio_sensor_custom
Connections:
- new net: SW2.4 (A), U3.8 (3V3)
- new net: BT2.1 (+), SW2.5 (B)
- new net: BT2.2 (-), U3.10 (GND)
Other:
- moved on the sheet: A1, BT1, BZ1, D1, J1, J2, J3, R1, R2, SW1, U1, U2

Commit message: journal 9, added S3 watch PCB, files
Parts:
- BZ3: footprint (none) -> Buzzer_Beeper:MagneticBuzzer_Kingstate_KCG0601
- J5: footprint ScottoKeebs_Components:OLED_128x64 -> ScottoKeebs_Scotto:OLED_128x64
- SW3, SW4, SW5, SW6: footprint (none) -> Button_Switch_THT:SW_PUSH_1P1T_6x3.5mm_H4.3_APEM_MJTP1243
Connections:
- net at BZ3.1 (+): now also U3.4 (SCK/D5)
- net at BZ3.2 (-): now also BT2.2 (-), BZ2.2 (-), D2.2 (GND), J5.1 (GND), SW3.2, SW4.2, SW5.2, SW6.2, U3.10 (GND)
- net at SW5.1: now also U3.7 (CS/D8)
- net at D2.4 (DIN): now also U3.6 (MOSI/D7)
- net at SW6.1: now also U3.12 (D3)
- net at SW2.4 (A), U3.8 (3V3): now also J5.2 (VCC)
- net at BZ2.1 (+): now also U3.5 (MISO/D6)
- net at SW3.1: now also U3.3 (D0)
- net at J5.3 (SCL): now also U3.14 (SCL/D1)
- net at J5.4 (SDA): now also U3.13 (SDA/D2)
- net at U3.11 (D4): now also SW4.1
Other:
- moved on the sheet: SW4, SW5, SW6
